File: Eagle/ChargerBase.brd (EAGLE design)
At the start: 32.7 x 23.5 mm, 14 parts, among them IC2 TINY24/44/84-SSU

Commit message: Updated uC code
Parts:
- removed PB1: PB1, switch-tact:DTSM-3
- removed PWM, PWR: (no value), adafruit:CHIPLED_0805
- removed R1, R3: (no value), rcl:R0805
- removed R4: 10K, rcl:R0805
- removed SV1, SV2: (no value), con-lstb:MA07-1
- removed U1: (no value), MicroUSB:USB-MICRO-SMD
- added CN1: (no value), adafruit:DCJACK_2MM_PTH
- added J1: (no value), con-jack:SPC4078
- added U$1: 2.1MMJACKTHM, adafruit:PJ-102A
- C1: value (none) -> 100n
- renumbered RST to NP
Connections:
- removed net N$1: PWR.A, R3.2
- removed net N$2: PWM.A, R1.2
- new net GNDBREAK: CN1.GNDBREAK
- new net PWR: CN1.PWR
- net GND: now also CN1.GND; no longer PB1.2, PWM.C, PWR.C, SV1.7, U1.GND1
- net MISO: no longer R1.1, SV1.1
- net MOSI: no longer SV2.7
- net N$3: no longer SV2.2
- net N$4: no longer SV2.3
- net N$5: no longer SV2.5
- net N$6: no longer SV2.6
- net PIN10: no longer SV1.3
- net PIN11: no longer SV1.4
- net PIN12: no longer SV1.5
- net PIN13: no longer PB1.1, R4.1, SV1.6
- net RST: no longer SV2.4
- net SCK: no longer SV1.2
- net VCC: no longer R3.1, R4.2, SV2.1, U1.VBUS1
Routing:
- net VCC: track 51.0 -> 36.5 mm
- net PIN13: track 23.1 -> 12.8 mm
- net MISO: track 16.3 -> 7.62 mm
- net RST: track 42.1 -> 34.5 mm
- net PIN11: track 6.29 -> 0.00 mm
- net MOSI: track 19.7 -> 14.3 mm
- net N$1: track 4.98 -> 0.00 mm
- net N$2: track 3.85 -> 0.00 mm
- net SCK: track 15.5 -> 12.0 mm
- net N$6: track 8.61 -> 5.02 mm
- net N$3: track 8.61 -> 5.02 mm
- net PIN12: track 6.81 -> 5.02 mm
- net PIN10: track 6.81 -> 5.02 mm
- net N$5: track 8.08 -> 6.29 mm
- net N$4: track 8.08 -> 6.29 mm

Commit message: Updated schematic
Parts:
- removed CN1: (no value), adafruit:DCJACK_2MM_PTH
- removed J1: (no value), con-jack:SPC4078
- added BARREL_JACK_2.1MM: (no value), adafruit:DCJACK_2MM_PTH
- added C2: (no value), adafruit:C025-040X050
- added C3, C4, C5, C6, C9: 1nF, rcl:C0805
- added C7, C8: (no value), adafruit:C050-025X075
- added D1, D2: 1N4004, adafruit:DO41-10
- added F1: 2A, special:FUSE
- added IC1, IC3: NE5532D, linear:SO08
- added L1: 47uH, rcl:0207/7
- added LED1, LED2, LED3, LED4, LED5: (no value), led:CHIPLED_0805
- added Q1, Q2, Q3: 2N3906, transistor-pnp:TO92
- added R1, R3, R4, R5, R6, R7, R8, R9: 1k, rcl:R0805
- added R10: 470, rcl:R0805
- added R11, R12, R13, R14, R15, R16: 1R, rcl:R0805
- added S1, S2: REED-SWITCH-CT10-1530-G1, switch-reed:CT10-G1
- added T1, T2, T3, T4: 2N3904, transistor:TO92
- added TX_COIL: 22-23-2021, con-molex:22-23-2021
- U$1: value 2.1MMJACKTHM -> AP1509; device adafruit:PJ-102A -> _VMS:SOP08
- moved U$1 5.39 mm to (-10.2, -5.08)
Connections:
- removed net GNDBREAK: CN1.GNDBREAK
- removed net PWR: CN1.PWR
- new net COIL_DRIVER: C6.2, C9.1, IC3.7, R6.1
- new net N$1: C3.1, IC1.3, R1.1, R3.2
- new net N$10: C4.2, IC1.7, R4.1, R8.2
- new net N$11: C5.1, IC3.3, R5.2, R8.1
- new net N$12: C5.2, IC3.1, R5.1, R9.2
- new net N$13: C6.1, IC3.5, R6.2, R9.1
- new net N$15: R12.2, T3.3
- new net N$16: R10.1
- new net N$17: LED1.C, LED2.A
- new net N$18: LED2.C, LED3.A
- new net N$19: LED3.C, LED4.A
- new net N$2: L1.1, U$1.2
- new net N$20: LED4.C, LED5.A
- new net N$21: LED5.C, R10.2
- new net N$22: S1.2, S2.1
- new net N$23: R13.2, T4.3
- new net N$24: Q1.3, R14.1
- new net N$25: Q2.3, R15.1
- new net N$26: Q3.3, R16.1
- new net N$27: C7.1, R11.1, R12.1, R13.1, R14.2, R15.2, R16.2
- new net N$28: C9.2, D1.A, T2.2, T3.2, T4.2
- new net N$29: D1.C, D2.A
- new net N$30: C7.2, C8.1, TX_COIL.1
- new net N$31: D2.C, Q1.2, Q2.2, Q3.2
- new net N$7: BARREL_JACK_2.1MM.PWR, F1.1
- new net N$8: IC1.1, R3.1, R7.2
- new net N$9: C4.1, IC1.5, R4.2, R7.1
- new net PWM: IC2.6, R1.2
- new net V+: IC1.8, IC3.8
- new net V-: IC1.4, IC3.4
- new net VDD: F1.2, LED1.A, T2.1, T3.1, T4.1, U$1.1
- net GND: now also BARREL_JACK_2.1MM.GND, BARREL_JACK_2.1MM.GNDBREAK, C2.2, C8.2, IC1.2, IC1.6, IC3.2, Q1.1, Q2.1, Q3.1, S2.2, T1.3, TX_COIL.2, U$1.4, U$1.5, U$1.6, U$1.7, U$1.8; no longer CN1.GND
- net N$6: now also R11.2, T2.3; no longer IC2.6
- net PIN12: now also S1.1
- net VCC: now also C2.1, L1.2, U$1.3
Routing:
- net PWM: track 0.00 -> 5.02 mm
- net N$6: track 5.02 -> 0.00 mm

Commit message: Uploaded schematics
Parts:
- removed D2: 1N4004, adafruit:DO41-10
- removed Q3: 2N3906, transistor-pnp:TO92
- removed R13, R14, R15, R16: 1R, rcl:R0805
- removed T4: 2N3904, transistor:TO92
- added LED10, LED6, LED7, LED8, LED9: (no value), led:CHIPLED_0805
- added R17: 1k, rcl:R0805
- added R18, R19: 10k, rcl:R0805
- added TM1: 100k, adafruit:TC33X
- C2: value (none) -> 10uF
- C7: value (none) -> 1uF
- C8: value (none) -> 10nF
- C9: value 1nF -> 100n
- Q2: value 2N3906 -> 1MHz; device transistor-pnp:TO92 -> adafruit:SM49
- R11: value 1R -> 470
- R12: value 1R -> 1k
- moved T3 142.9 mm to (-76.2, -288.3)
- moved R11 105.2 mm to (-77.5, -275.6)
- moved Q2 102.0 mm to (-71.1, -262.9)
- moved R12 92.0 mm to (-72.4, -269.2)
- moved IC1 58.5 mm to (27.9, 5.08)
- moved U$1 44.0 mm to (26.7, 19.1)
Connections:
- removed net N$23: R13.2, T4.3
- removed net PIN10: IC2.10
- removed net PIN11: IC2.11
- removed net V+: IC1.8, IC3.8
- removed net V-: IC1.4, IC3.4
- new net LED1: IC2.10, R12.2
- new net LED2: IC2.11, R17.2
- new net N$14: R17.1, T1.2
- new net N$32: R11.1, T3.1
- new net N$33: R12.1, T3.2
- net GND: now also IC1.4, IC3.4, R19.1, T3.3, TM1.1; no longer Q2.1, Q3.1
- net N$15: now also IC3.6, TM1.2; no longer R12.2, T3.3
- net N$16: now also T1.1
- net N$24: now also LED7.C, LED8.A; no longer Q1.3, R14.1
- net N$25: now also LED8.C, LED9.A; no longer Q2.3, R15.1
- net N$26: now also LED10.A, LED9.C; no longer Q3.3, R16.1
- net N$27: now also Q1.3, T2.3; no longer R11.1, R12.1, R13.1, R14.2, R15.2, R16.2
- net N$28: now also R18.1; no longer T3.2, T4.2
- net N$29: now also Q1.2, R19.2; no longer D2.A
- net N$3: now also Q2.1
- net N$31: now also LED10.C, R11.2; no longer D2.C, Q1.2, Q2.2, Q3.2
- net N$4: now also Q2.2
- net N$6: now also LED6.C, LED7.A; no longer R11.2, T2.3
- net N$8: now also C3.2
- net VDD: now also IC1.8, IC3.8, LED6.A, R18.2, TM1.3; no longer T3.1, T4.1
Routing:
- net VDD: track 0.00 -> 8.77 mm
- net GND: track 0.00 -> 8.77 mm
- net PIN10: track 5.02 -> 0.00 mm
- net LED1: track 0.00 -> 5.02 mm
- removed copper zone on layer 1, net GND
