File: Eagle/ChargerBase.sch (EAGLE design)
At the start: 8 parts, among them IC2 TINY24/44/84-SSU

Commit message: Updated schematic
Parts:
- removed CN1: (no value), adafruit:DCBARRELPTH
- removed J1: (no value), con-jack:JACK-PLUG1
- added BARREL_JACK_2.1MM: (no value), adafruit:DCBARRELPTH
- added C2: (no value), adafruit:C-US025-040X050
- added C3, C4, C5, C6, C9: 1nF, rcl:C-EUC0805
- added C7, C8: (no value), adafruit:C-US050-025X075
- added D1, D2: 1N4004, adafruit:1N4004
- added F1: 2A, special:FUSE
- added IC1, IC3: NE5532D, linear:NE5532D
- added L1: 47uH, rcl:L-US0207/7
- added LED1, LED2, LED3, LED4, LED5: (no value), led:LEDCHIPLED_0805
- added Q1, Q2, Q3: 2N3906, transistor-pnp:2N3906
- added R1, R3, R4, R5, R6, R7, R8, R9: 1k, rcl:R-US_R0805
- added R10: 470, rcl:R-US_R0805
- added R11, R12, R13, R14, R15, R16: 1R, rcl:R-US_R0805
- added S1, S2: REED-SWITCH-CT10-1530-G1, switch-reed:REED-SWITCH-CT10-1530-G1
- added T1, T2, T3, T4: 2N3904, transistor:2N3904
- added TX_COIL: 22-23-2021, con-molex:22-23-2021
- U$1: value 2.1MMJACKTHM -> AP1509; device adafruit:2.1MMJACKTHM -> _VMS:AP1509
Connections:
- new net COIL_DRIVER: C6.2, C9.1, IC3B.OUT, R6.1
- new net N$1: C3.1, IC1A.+IN, R1.1, R3.2
- new net N$10: C4.2, IC1B.OUT, R4.1, R8.2
- new net N$11: C5.1, IC3A.+IN, R5.2, R8.1
- new net N$12: C5.2, IC3A.OUT, R5.1, R9.2
- new net N$13: C6.1, IC3B.+IN, R6.2, R9.1
- new net N$15: R12.2, T3.E
- new net N$16: R10.1
- new net N$17: LED1.C, LED2.A
- new net N$18: LED2.C, LED3.A
- new net N$19: LED3.C, LED4.A
- new net N$2: L1.1, U$1.OUT
- new net N$20: LED4.C, LED5.A
- new net N$21: LED5.C, R10.2
- new net N$22: S1.2, S2.1
- new net N$23: R13.2, T4.E
- new net N$24: Q1.E, R14.1
- new net N$25: Q2.E, R15.1
- new net N$26: Q3.E, R16.1
- new net N$27: C7.1, R11.1, R12.1, R13.1, R14.2, R15.2, R16.2
- new net N$28: C9.2, D1.A, T2.B, T3.B, T4.B
- new net N$29: D1.C, D2.A
- new net N$30: C7.2, C8.1, TX_COIL-1.S
- new net N$31: D2.C, Q1.B, Q2.B, Q3.B
- new net N$7: BARREL_JACK_2.1MM.PWR, F1.1
- new net N$8: IC1A.OUT, R3.1, R7.2
- new net N$9: C4.1, IC1B.+IN, R4.2, R7.1
- new net PWM: IC2.(PCINT7/ICP/OC0B/ADC7)PA7, R1.2
- new net VDD: F1.2, LED1.A, T2.C, T3.C, T4.C, U$1.VIN
- net GND: now also BARREL_JACK_2.1MM.GND, BARREL_JACK_2.1MM.GNDBREAK, C2.2, C8.2, IC1A.-IN, IC1B.-IN, IC3A.-IN, Q1.C, Q2.C, Q3.C, S2.2, T1.E, TX_COIL-2.S, U$1.GND5, U$1.GND6, U$1.GND7, U$1.GND8, U$1.SD
- net N$6: now also R11.2, T2.E; no longer IC2.(PCINT7/ICP/OC0B/ADC7)PA7
- net PIN12: now also S1.1
- net VCC: now also C2.1, L1.2, U$1.FB
Other:
- note added: "12VDC in, 12/5V out"
- note added: "Coil Driving Stage"
- note added: "Filtering"
- note added: "Offset and Gain"
- note added: "Signal conditioning stage"
- moved on the sheet: C1, IC2, ISP1, NP, R2

Commit message: Uploaded schematics
Parts:
- removed D2: 1N4004, adafruit:1N4004
- removed Q3: 2N3906, transistor-pnp:2N3906
- removed R13, R14, R15, R16: 1R, rcl:R-US_R0805
- removed T4: 2N3904, transistor:2N3904
- added LED10, LED6, LED7, LED8, LED9: (no value), led:LEDCHIPLED_0805
- added R17: 1k, rcl:R-US_R0805
- added R18, R19: 10k, rcl:R-US_R0805
- added TM1: 100k, adafruit:TRIMPOTTC33X
- C2: value (none) -> 10uF
- C7: value (none) -> 1uF
- C8: value (none) -> 10nF
- C9: value 1nF -> 100n
- Q2: value 2N3906 -> 1MHz; device transistor-pnp:2N3906 -> adafruit:CRYSTALSM49
- R11: value 1R -> 470
- R12: value 1R -> 1k
Connections:
- removed net N$23: R13.2, T4.E
- removed net PIN10: IC2.(PCINT3/T0/ADC3)PA3
- removed net PIN11: IC2.(PCINT2/AIN1/ADC2)PA2
- new net LED1: IC2.(PCINT3/T0/ADC3)PA3, R12.2
- new net LED2: IC2.(PCINT2/AIN1/ADC2)PA2, R17.2
- new net N$14: R17.1, T1.B
- new net N$32: R11.1, T3.C
- new net N$33: R12.1, T3.B
- net GND: now also IC1P.V-, IC3P.V-, R19.1, T3.E, TM1.A; no longer Q2.C, Q3.C
- net N$15: now also IC3B.-IN, TM1.S; no longer R12.2, T3.E
- net N$16: now also T1.C
- net N$24: now also LED7.C, LED8.A; no longer Q1.E, R14.1
- net N$25: now also LED8.C, LED9.A; no longer Q2.E, R15.1
- net N$26: now also LED10.A, LED9.C; no longer Q3.E, R16.1
- net N$27: now also Q1.E, T2.E; no longer R11.1, R12.1, R13.1, R14.2, R15.2, R16.2
- net N$28: now also R18.1; no longer T3.B, T4.B
- net N$29: now also Q1.B, R19.2; no longer D2.A
- net N$3: now also Q2.1
- net N$31: now also LED10.C, R11.2; no longer D2.C, Q1.B, Q2.B, Q3.B
- net N$4: now also Q2.2
- net N$6: now also LED6.C, LED7.A; no longer R11.2, T2.E
- net N$8: now also C3.2
- net VDD: now also IC1P.V+, IC3P.V+, LED6.A, R18.2, TM1.E; no longer T3.C, T4.C
Other:
- note added: "Placement indicator LEDs"
- moved on the sheet: C1, C3, C4, C5, C6, C7, C8, C9, D1, IC1A, IC1B, IC2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
