File: Eagle/T10_ChargerBase.brd (EAGLE design)
At the start: 32.7 x 23.5 mm, 53 parts, among them IC1 NE5532D, IC2 TINY24/44/84-SSU, IC3 NE5532D, Q1 2N3906, Q2 1MHz, T1 2N3904, T2 2N3904, T3 2N3904

Commit message: Board files and update uC program
Parts:
- removed F1: 2A, special:FUSE
- removed L1: 47uH, rcl:0207/7
- removed LED1, LED6: (no value), led:CHIPLED_0805
- removed NP: RST, switch-tact:DTSM-3
- removed Q2: 1MHz, adafruit:SM49
- added C10, C11: (no value), adafruit:E2-5
- added C12: 100n, rcl:C0805
- added IC5: AZ1117IH-5.0V, _VMS:SOT223
- C2: value 10uF -> 100n; device adafruit:C025-040X050 -> rcl:C0805
- S1, S2: value REED-SWITCH-CT10-1530-G1 -> REED-SWITCH-MK6-6; device switch-reed:CT10-G1 -> switch-reed:MK6-6
- U$1: value AP1509 -> LITTLEFUSE; device _VMS:SOP08 -> _VMS:LITTLEFUSE
- moved T3 375.2 mm to (35.6, 69.8), turned to 180 degrees
- moved R11 368.5 mm to (40.0, 73.7), turned to 90 degrees
- moved LED10 366.3 mm to (40.0, 76.8), turned to 90 degrees
- moved LED7 361.1 mm to (3.81, 77.5), turned to 180 degrees
- moved R12 348.6 mm to (39.4, 61.0), turned to 180 degrees
- moved R17 326.2 mm to (29.2, 68.6), turned to 180 degrees
- moved TM1 313.4 mm to (30.5, 39.4)
- moved LED9 308.2 mm to (41.1, 3.81)
- moved LED8 298.1 mm to (2.54, 4.32), turned to 180 degrees
- moved R19 293.6 mm to (21.6, 24.1)
- moved C9 286.0 mm to (27.9, 33.0), turned to 270 degrees
- moved R18 285.3 mm to (14.0, 24.1)
- moved C8 252.6 mm to (17.8, 8.89), turned to 180 degrees
- moved C7 252.6 mm to (17.8, 14.0), turned to 270 degrees
- moved TX_COIL 246.7 mm to (17.8, 5.08), turned to 180 degrees
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Connections:
- removed net N$17 (its old number): LED1.C, LED2.A
- removed net N$2 (its old number): L1.1, U$1.2
- removed net N$6 (its old number): LED6.C, LED7.A
- net GND: now also C10.-, C11.-, C12.2, IC5.1; no longer NP.2, U$1.4, U$1.5, U$1.6, U$1.7, U$1.8
- net N$3: no longer Q2.1
- net N$4: no longer Q2.2
- net N$7: now also U$1.1; no longer F1.1
- net RST: no longer NP.1
- net VCC: now also C10.+, IC5.4; no longer C2.1, L1.2, U$1.3
- net VDD: now also C11.+, C12.1, C2.1, IC5.3, LED2.A, LED7.A, U$1.2; no longer F1.2, LED1.A, LED6.A, U$1.1
Routing:
- net GND: track 8.77 -> 286.7 mm, vias 0 -> 5
- net VDD: track 8.77 -> 208.1 mm, vias 0 -> 6
- net N$20: track 0.00 -> 78.4 mm
- net N$18: track 0.00 -> 73.9 mm
- net N$26: track 0.00 -> 73.6 mm
- net N$24: track 0.00 -> 73.2 mm
- net PIN12: track 5.02 -> 59.5 mm, vias 0 -> 1
- net N$19: track 0.00 -> 42.8 mm
- net PWM: track 5.02 -> 45.4 mm, vias 0 -> 2
- net N$25: track 0.00 -> 40.2 mm
- net N$11: track 0.00 -> 33.3 mm, vias 0 -> 2
- net N$28: track 0.00 -> 30.1 mm
- net N$22: track 0.00 -> 26.7 mm
- net N$13: track 0.00 -> 23.5 mm, vias 0 -> 2
- net N$8: track 0.00 -> 20.7 mm
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- removed copper zone on layer 16, net GND
Other:
- board size 32.7 x 23.5 mm -> 44.6 x 80.3 mm
