File: Eagle/T10_ChargerBase.sch (EAGLE design)
At the start: 53 parts, among them IC1 NE5532D, IC2 TINY24/44/84-SSU, IC3 NE5532D, Q1 2N3906, Q2 1MHz, T1 2N3904, T2 2N3904, T3 2N3904

Commit message: Board files and update uC program
Parts:
- removed F1: 2A, special:FUSE
- removed L1: 47uH, rcl:L-US0207/7
- removed LED1, LED6: (no value), led:LEDCHIPLED_0805
- removed NP: RST, switch-tact:DTSM-3
- removed Q2: 1MHz, adafruit:CRYSTALSM49
- added C10, C11: (no value), adafruit:CPOL-USE2-5
- added C12: 100n, rcl:C-USC0805
- added IC5: AZ1117IH-5.0V, _VMS:317EMP
- C2: value 10uF -> 100n; device adafruit:C-US025-040X050 -> rcl:C-USC0805
- S1, S2: value REED-SWITCH-CT10-1530-G1 -> REED-SWITCH-MK6-6; device switch-reed:REED-SWITCH-CT10-1530-G1 -> switch-reed:REED-SWITCH-MK6-6
- U$1: value AP1509 -> LITTLEFUSE; device _VMS:AP1509 -> _VMS:LITTLEFUSE
Connections:
- removed net N$17 (its old number): LED1.C, LED2.A
- removed net N$2 (its old number): L1.1, U$1.OUT
- removed net N$6 (its old number): LED6.C, LED7.A
- net GND: now also C10.-, C11.-, C12.2, IC5.ADJ; no longer NP.2, U$1.GND5, U$1.GND6, U$1.GND7, U$1.GND8, U$1.SD
- net N$3: no longer Q2.1
- net N$4: no longer Q2.2
- net N$7: now also U$1.P$1; no longer F1.1
- net RST: no longer NP.1
- net VCC: now also C10.+, IC5.VO; no longer C2.1, L1.2, U$1.FB
- net VDD: now also C11.+, C12.1, C2.1, IC5.VI, LED2.A, LED7.A, U$1.P$2; no longer F1.2, LED1.A, LED6.A, U$1.VIN
Other:
- moved on the sheet: BARREL_JACK_2.1MM, C2, LED10, R11, R12, R17, T3
