File: Eagle/T10_Receiver.sch (EAGLE design)
At the start: 9 parts, among them X1 22-23-2021, X2 22-23-2021

Commit message: Board files and update uC program
Parts:
- removed C1: 10uF, rcl:C-EU025-030X050
- removed C2: 10nF, rcl:C-EU025-030X050
- added C3, C4, C5: (no value), adafruit:C-USC0805
Connections:
- net N$1: now also C3.1; no longer C2.1
- net N$2: now also C3.2; no longer C2.2
- net N$3: now also C4.2, C5.2; no longer C1.2
- net N$4: now also C4.1, C5.1; no longer C1.1
