File: Eagle/ece411-t10-ChargerBase.brd (EAGLE design)
At the start: 40.8 x 43.4 mm, 33 parts, among them IC2 TINY24/44/84-SSU, IC5 AZ1117IH-5.0V, Q1-NP NP, Q2-NP NP, Q3-NP NP, Q4 NP, Q5-NP NP, Q6 RFD16N05LSM9ACTTO252, T1 2N3904, T3 2N3904

Commit message: cleaned up schematic. fixed minor ERC error
Parts:
- C10, C11: value (none) -> 10u
- LED10, LED7, LED8, LED9: value (none) -> green
- LED2, LED3, LED4, LED5: value (none) -> red
Connections:
- removed net N$3: IC2.2
- removed net N$4: IC2.3
- removed net N$5: IC2.5
- removed net PIN13: IC2.13
Changed lines of the file:
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@@
 <element name="IC2" library="avr-5" package="SOIC14" value="TINY24/44/84-SSU" x="27.94" y="62.23"/>
 <element name="ISP1" library="adafruit" package="AVRISP" value="AVRISP-6" x="15.24" y="59.69" rot="R180"/>
-<element name="LED10" library="led" package="CHIPLED_0805" value="" x="36.703" y="77.089" rot="R90"/>
-<element name="LED2" library="led" package="CHIPLED_0805" value="" x="1.27" y="77.47" smashed="yes" rot="R180">
+<element name="LED10" library="led" package="CHIPLED_0805" value="green" x="36.703" y="77.089" rot="R90"/>
+<element name="LED2" library="led" package="CHIPLED_0805" value="red" x="1.27" y="77.47" smashed="yes" rot="R180">
 <attribute name="NAME" x="0.508" y="75.184" size="1.27" layer="25" rot="R270"/>
 <attribute name="VALUE" x="-1.27" y="78.74" size="1.27" layer="27" rot="R270"/>
 </element>
-<element name="LED3" library="led" package="CHIPLED_0805" value="" x="1.016" y="38.862" smashed="yes" rot="R180">
+<element name="LED3" library="led" package="CHIPLED_0805" value="red" x="1.016" y="38.862" smashed="yes" rot="R180">
 <attribute name="NAME" x="0.254" y="45.466" size="1.27" layer="25" rot="R270"/>
 <attribute name="VALUE" x="-1.524" y="40.132" size="1.27" layer="27" rot="R270"/>
 </element>
-<element name="LED4" library="led" package="CHIPLED_0805" value="" x="38.1" y="38.1" smashed="yes" rot="R270">
+<element name="LED4" library="led" package="CHIPLED_0805" value="red" x="38.1" y="38.1" smashed="yes" rot="R270">
 <attribute name="NAME" x="32.004" y="37.084" size="1.27" layer="25"/>
 <attribute name="VALUE" x="36.83" y="35.56" size="1.27" layer="27"/>
 </element>
-<element name="LED5" library="led" package="CHIPLED_0805" value="" x="38.1" y="78.74" rot="R90"/>
-<element name="LED7" library="led" package="CHIPLED_0805" value="" x="3.81" y="77.47" rot="R180"/>
-<element name="LED8" library="led" package="CHIPLED_0805" value="" x="2.54" y="41.148" smashed="yes" rot="R180">
+<element name="LED5" library="led" package="CHIPLED_0805" value="red" x="38.1" y="78.74" rot="R90"/>
+<element name="LED7" library="led" package="CHIPLED_0805" value="green" x="3.81" y="77.47" rot="R180"/>
+<element name="LED8" library="led" package="CHIPLED_0805" value="green" x="2.54" y="41.148" smashed="yes" rot="R180">
 <attribute name="NAME" x="1.778" y="47.498" size="1.27" layer="25" rot="R270"/>
 <attribute name="VALUE" x="0" y="42.418" size="1.27" layer="27" rot="R270"/>
 </element>
-<element name="LED9" library="led" package="CHIPLED_0805" value="" x="36.83" y="40.132" smashed="yes" rot="R270">
+<element name="LED9" library="led" package="CHIPLED_0805" value="green" x="36.83" y="40.132" smashed="yes" rot="R270">
 <attribute name="NAME" x="39.878" y="39.37" size="1.27" layer="25" rot="R90"/>
 <attribute name="VALUE" x="35.56" y="37.592" size="1.27" layer="27"/>
@@
 </element>
 <element name="U$1" library="_VMS" package="LITTLEFUSE" value="LITTLEFUSE" x="3.81" y="66.04" rot="R270"/>
-<element name="C11" library="adafruit" package="E2-5" value="" x="8.89" y="62.23"/>
-<element name="C10" library="adafruit" package="E2-5" value="" x="21.59" y="74.93"/>
+<element name="C11" library="adafruit" package="E2-5" value="10u" x="8.89" y="62.23"/>
+<element name="C10" library="adafruit" package="E2-5" value="10u" x="21.59" y="74.93"/>
 <element name="IC5" library="_VMS" package="SOT223" value="AZ1117IH-5.0V" x="27.94" y="74.93"/>
 <element name="Q1-NP" library="transistor-fet" package="TO-92" value="NP" x="26.67" y="52.07" smashed="yes" rot="R180">
@@
 <wire x1="8.448" y1="58.166" x2="8.382" y2="58.1" width="0.6096" layer="1"/>
 </signal>
-<signal name="N$3">
-<contactref element="IC2" pad="2"/>
-</signal>
-<signal name="N$4">
-<contactref element="IC2" pad="3"/>
-</signal>
-<signal name="N$5">
-<contactref element="IC2" pad="5"/>
-</signal>
 <signal name="PWM">
 <contactref element="Q3-NP" pad="2"/>
@@
 <wire x1="26.67" y1="68.58" x2="26.67" y2="64.8335" width="0.6096" layer="1"/>
 </signal>
-<signal name="PIN13">
-<contactref element="IC2" pad="13"/>
-</signal>
 <signal name="VDD">

Commit message: clean up
Parts:
- moved BARREL_JACK_2.1MM 7.94 mm to (13.5, 73.4), turned to 0 degrees
Connections:
- net VCC: now also IC5.2
Routing:
- net GND: track 132.4 -> 124.3 mm, vias 2 -> 12
- net VCC: track 44.1 -> 51.5 mm
- net N$7: track 17.0 -> 19.1 mm
- net VDD: track 103.2 -> 105.1 mm
Other:
- board text removed: "I love lamp"
