File: Eagle/ece411-t10-Receiver.brd (EAGLE design)
At the start: 10.6 x 19.8 mm, 12 parts, among them X1 22-23-2021, X3 USB

Commit message: clean up
Connections:
- net N$4 renamed 5V
- net N$8 renamed GND
