File: Eagle/ece411-t10-Receiver.sch (EAGLE design)
At the start: 10 parts, among them X1 22-23-2021, X2 22-23-2021

Commit message: Boards + schematics rev2
Parts:
- removed C4, C5: (no value), adafruit:C-USC0805
- removed D1, D2, D3, D4: DFLS230LQ-7, adafruit:DIODESOD-523
- removed X2: 22-23-2021, con-molex:22-23-2021
- added C1: 100n+, adafruit:C-USC0805
- added C2: 100n, adafruit:C-USC0805
- added R1: 75k, resistor:R-US_R0805
- added R2: 51k, resistor:R-US_R0805
- added U$1, U$2, U$3, U$4: DFLS230LQ-SCHOTTKY, _VMS:DFLS230LQ-SCHOTTKY
- added X3: USB, con-molex:22-23-2041
- C3: value (none) -> NP
- D5: value 5.1V -> DZ2405100LCT-ZENER; device diode:BZX84CSMD -> _VMS:DZ2405100LCT-ZENER
Connections:
- removed net N$3: C4.2, C5.2, D1.A, D2.A, D5.A, X2-2.S
- new net N$5: R1.1, R2.2, X3-2.S, X3-3.S
- new net N$8: C1.2, C2.2, D5.A, R2.1, U$1.A, U$3.A, X3-4.S
- net N$1: now also U$1.C, U$2.A; no longer D1.C, D3.A
- net N$2: now also U$3.C, U$4.A; no longer D2.C, D4.A
- net N$4: now also C1.1, C2.1, R1.2, U$2.C, U$4.C, X3-1.S; no longer C4.1, C5.1, D3.C, D4.C, X2-1.S
Other:
- moved on the sheet: X1-1, X1-2

Commit message: IO working on program
Other:
- note added: "+5V"
- note added: "D+"
- note added: "D-"
- note added: "GND"
- note added: "To Coil. ~20uH"
Changed lines of the file:
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@@
 <sheet>
 <plain>
+<text x="76.2" y="101.6" size="2.54" layer="97" rot="R180">To Coil. ~20uH</text>
+<wire x1="83.82" y1="106.68" x2="66.04" y2="106.68" width="0.1524" layer="97"/>
+<wire x1="66.04" y1="104.14" x2="66.04" y2="106.68" width="0.1524" layer="97" curve="-180"/>
+<wire x1="66.04" y1="101.6" x2="66.04" y2="104.14" width="0.1524" layer="97" curve="-180"/>
+<wire x1="66.04" y1="99.06" x2="66.04" y2="101.6" width="0.1524" layer="97" curve="-180"/>
+<wire x1="66.04" y1="96.52" x2="66.04" y2="99.06" width="0.1524" layer="97" curve="-180"/>
+<wire x1="66.04" y1="93.98" x2="66.04" y2="96.52" width="0.1524" layer="97" curve="-180"/>
+<wire x1="66.04" y1="93.98" x2="83.82" y2="93.98" width="0.1524" layer="97"/>
+<text x="205.74" y="114.3" size="2.54" layer="97" rot="R180">+5V</text>
+<text x="205.74" y="88.9" size="2.54" layer="97" rot="R180">GND</text>
+<text x="205.74" y="104.14" size="2.54" layer="97" rot="R180">D-</text>
+<text x="205.74" y="96.52" size="2.54" layer="97" rot="R180">D+</text>
 </plain>
 <instances>

Commit message: clean up
Connections:
- net N$4 renamed 5V
- net N$8 renamed GND
Changed lines of the file:
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@@
 </segment>
 </net>
-<net name="N$4" class="0">
+<net name="5V" class="0">
 <segment>
 <wire x1="139.7" y1="111.76" x2="139.7" y2="109.22" width="0.1524" layer="91"/>
@@
 </segment>
 </net>
-<net name="N$8" class="0">
+<net name="GND" class="0">
 <segment>
 <pinref part="U$1" gate="G$1" pin="A"/>
